Commit message: Shrink all arm scaffolds to fit under the x500 landing gear
Observation in Gazebo: the arm tip punched through the ground before
the landing gear feet touched down. Measurements:
  x500 gear feet at z = -0.2195 m below base_link
  three_dof arm drop  = 0.05 + 0.12 + 0.12 + 0.072 + 0.015 = 0.377 m
                        (16 cm past the gear)
  scaffold arms drop more (panda 7 x 0.10, ur5 6 x 0.12, ...)

Rule the arm to fit: total drop budget = 0.20 m
  = 0.05 m mount offset
  + N * link_len (chosen so N * link_len ~ 0.13 m)
  + 0.015 m end-effector sphere

New segment lengths per arm:
  three_dof:    3 x 0.040 m  -> 0.185 m drop (+34 mm above feet)
  openmanip_x:  4 x 0.033 m  -> 0.197 m drop (+22 mm above feet)
  panda:        7 x 0.019 m  -> 0.198 m drop (+21 mm above feet)
  ur5:          6 x 0.022 m  -> 0.197 m drop (+22 mm above feet)

Inertias, radii, and visual cylinder lengths were scaled to match.
arms/three_dof/urdf/three_dof.urdf.xacro: link_len 0.12 -> 0.04,
link_radius 0.012 -> 0.008. Same SDF dimensions in the composed model.
Generator script /tmp/gen_arm_scaffolds.py regenerated the other three.

Pytest: 42 passing.

File: arms/openmanip_x/urdf/openmanip_x.urdf.xacro (robot description, xacro)
@@ -9,17 +9,17 @@
     <link name="${name}">
       <inertial>
-        <mass value="0.1"/>
-        <origin xyz="0 0 0.0500" rpy="0 0 0"/>
-        <inertia ixx="8.693333e-05" iyy="8.693333e-05" izz="7.200000e-06"
+        <mass value="0.04"/>
+        <origin xyz="0 0 0.0165" rpy="0 0 0"/>
+        <inertia ixx="4.270000e-06" iyy="4.270000e-06" izz="1.280000e-06"
                  ixy="0" ixz="0" iyz="0"/>
       </inertial>
       <visual>
-        <origin xyz="0 0 0.0500" rpy="0 0 0"/>
-        <geometry><cylinder radius="0.012" length="0.1"/></geometry>
+        <origin xyz="0 0 0.0165" rpy="0 0 0"/>
+        <geometry><cylinder radius="0.008" length="0.033"/></geometry>
         <material name="${name}_mat"><color rgba="${color_r} ${color_g} ${color_b} 1"/></material>
       </visual>
       <collision>
-        <origin xyz="0 0 0.0500" rpy="0 0 0"/>
-        <geometry><cylinder radius="0.012" length="0.1"/></geometry>
+        <origin xyz="0 0 0.0165" rpy="0 0 0"/>
+        <geometry><cylinder radius="0.008" length="0.033"/></geometry>
       </collision>
     </link>
@@ -39,5 +39,5 @@
     <parent link="openmanip_x_link1"/>
     <child link="openmanip_x_link2"/>
-    <origin xyz="0 0 0.1000" rpy="0 0 0"/>
+    <origin xyz="0 0 0.0330" rpy="0 0 0"/>
     <axis xyz="0 1 0"/>
     <limit lower="-3.14159" upper="3.14159" effort="2.0" velocity="3.0"/>
@@ -48,5 +48,5 @@
     <parent link="openmanip_x_link2"/>
     <child link="openmanip_x_link3"/>
-    <origin xyz="0 0 0.1000" rpy="0 0 0"/>
+    <origin xyz="0 0 0.0330" rpy="0 0 0"/>
     <axis xyz="0 1 0"/>
     <limit lower="-3.14159" upper="3.14159" effort="2.0" velocity="3.0"/>
@@ -57,5 +57,5 @@
     <parent link="openmanip_x_link3"/>
     <child link="openmanip_x_link4"/>
-    <origin xyz="0 0 0.1000" rpy="0 0 0"/>
+    <origin xyz="0 0 0.0330" rpy="0 0 0"/>
     <axis xyz="0 1 0"/>
     <limit lower="-3.14159" upper="3.14159" effort="2.0" velocity="3.0"/>
@@ -76,5 +76,5 @@
     <parent link="openmanip_x_link4"/>
     <child link="end_effector_link"/>
-    <origin xyz="0 0 0.1100" rpy="0 0 0"/>
+    <origin xyz="0 0 0.0430" rpy="0 0 0"/>
   </joint>
   <xacro:arg name="sim_mode" default="gz"/>

File: arms/panda/urdf/panda.urdf.xacro (robot description, xacro)
@@ -9,17 +9,17 @@
     <link name="${name}">
       <inertial>
-        <mass value="0.3"/>
-        <origin xyz="0 0 0.0500" rpy="0 0 0"/>
-        <inertia ixx="2.692000e-04" iyy="2.692000e-04" izz="3.840000e-05"
+        <mass value="0.025"/>
+        <origin xyz="0 0 0.0095" rpy="0 0 0"/>
+        <inertia ixx="1.152083e-06" iyy="1.152083e-06" izz="8.000000e-07"
                  ixy="0" ixz="0" iyz="0"/>
       </inertial>
       <visual>
-        <origin xyz="0 0 0.0500" rpy="0 0 0"/>
-        <geometry><cylinder radius="0.016" length="0.1"/></geometry>
+        <origin xyz="0 0 0.0095" rpy="0 0 0"/>
+        <geometry><cylinder radius="0.008" length="0.019"/></geometry>
         <material name="${name}_mat"><color rgba="${color_r} ${color_g} ${color_b} 1"/></material>
       </visual>
       <collision>
-        <origin xyz="0 0 0.0500" rpy="0 0 0"/>
-        <geometry><cylinder radius="0.016" length="0.1"/></geometry>
+        <origin xyz="0 0 0.0095" rpy="0 0 0"/>
+        <geometry><cylinder radius="0.008" length="0.019"/></geometry>
       </collision>
     </link>
@@ -39,5 +39,5 @@
     <parent link="panda_link1"/>
     <child link="panda_link2"/>
-    <origin xyz="0 0 0.1000" rpy="0 0 0"/>
+    <origin xyz="0 0 0.0190" rpy="0 0 0"/>
     <axis xyz="0 1 0"/>
     <limit lower="-3.14159" upper="3.14159" effort="2.0" velocity="3.0"/>
@@ -48,5 +48,5 @@
     <parent link="panda_link2"/>
     <child link="panda_link3"/>
-    <origin xyz="0 0 0.1000" rpy="0 0 0"/>
+    <origin xyz="0 0 0.0190" rpy="0 0 0"/>
     <axis xyz="0 1 0"/>
     <limit lower="-3.14159" upper="3.14159" effort="2.0" velocity="3.0"/>
@@ -57,5 +57,5 @@
     <parent link="panda_link3"/>
     <child link="panda_link4"/>
-    <origin xyz="0 0 0.1000" rpy="0 0 0"/>
+    <origin xyz="0 0 0.0190" rpy="0 0 0"/>
     <axis xyz="0 1 0"/>
     <limit lower="-3.14159" upper="3.14159" effort="2.0" velocity="3.0"/>
@@ -66,5 +66,5 @@
     <parent link="panda_link4"/>
     <child link="panda_link5"/>
-    <origin xyz="0 0 0.1000" rpy="0 0 0"/>
+    <origin xyz="0 0 0.0190" rpy="0 0 0"/>
     <axis xyz="0 1 0"/>
     <limit lower="-3.14159" upper="3.14159" effort="2.0" velocity="3.0"/>
@@ -75,5 +75,5 @@
     <parent link="panda_link5"/>
     <child link="panda_link6"/>
-    <origin xyz="0 0 0.1000" rpy="0 0 0"/>
+    <origin xyz="0 0 0.0190" rpy="0 0 0"/>
     <axis xyz="0 1 0"/>
     <limit lower="-3.14159" upper="3.14159" effort="2.0" velocity="3.0"/>
@@ -84,5 +84,5 @@
     <parent link="panda_link6"/>
     <child link="panda_link7"/>
-    <origin xyz="0 0 0.1000" rpy="0 0 0"/>
+    <origin xyz="0 0 0.0190" rpy="0 0 0"/>
     <axis xyz="0 1 0"/>
     <limit lower="-3.14159" upper="3.14159" effort="2.0" velocity="3.0"/>
@@ -103,5 +103,5 @@
     <parent link="panda_link7"/>
     <child link="panda_hand"/>
-    <origin xyz="0 0 0.1100" rpy="0 0 0"/>
+    <origin xyz="0 0 0.0290" rpy="0 0 0"/>
   </joint>
   <xacro:arg name="sim_mode" default="gz"/>

File: arms/three_dof/urdf/three_dof.urdf.xacro (robot description, xacro)
@@ -9,7 +9,12 @@
 -->
 <robot xmlns:xacro="http://www.ros.org/wiki/xacro" name="three_dof">
+  <!--
+    Sizing: total drop below base_link must stay above the x500 landing
+    gear feet at z = -0.2195 m. Budget = 0.20 m total = 0.05 mount + 3
+    segments + 0.015 ee, so segments capped at 0.04 m.
+  -->
   <xacro:property name="density"     value="800.0"/>
-  <xacro:property name="link_len"    value="0.12"/>
-  <xacro:property name="link_radius" value="0.012"/>
+  <xacro:property name="link_len"    value="0.04"/>
+  <xacro:property name="link_radius" value="0.008"/>
   <xacro:property name="pi"          value="3.14159265359"/>
   <xacro:macro name="cyl_inertia" params="m r l">

File: arms/ur5/urdf/ur5.urdf.xacro (robot description, xacro)
@@ -9,17 +9,17 @@
     <link name="${name}">
       <inertial>
-        <mass value="0.4"/>
-        <origin xyz="0 0 0.0600" rpy="0 0 0"/>
-        <inertia ixx="5.124000e-04" iyy="5.124000e-04" izz="6.480000e-05"
+        <mass value="0.03"/>
+        <origin xyz="0 0 0.0110" rpy="0 0 0"/>
+        <inertia ixx="1.817500e-06" iyy="1.817500e-06" izz="1.215000e-06"
                  ixy="0" ixz="0" iyz="0"/>
       </inertial>
       <visual>
-        <origin xyz="0 0 0.0600" rpy="0 0 0"/>
-        <geometry><cylinder radius="0.018" length="0.12"/></geometry>
+        <origin xyz="0 0 0.0110" rpy="0 0 0"/>
+        <geometry><cylinder radius="0.009" length="0.022"/></geometry>
         <material name="${name}_mat"><color rgba="${color_r} ${color_g} ${color_b} 1"/></material>
       </visual>
       <collision>
-        <origin xyz="0 0 0.0600" rpy="0 0 0"/>
-        <geometry><cylinder radius="0.018" length="0.12"/></geometry>
+        <origin xyz="0 0 0.0110" rpy="0 0 0"/>
+        <geometry><cylinder radius="0.009" length="0.022"/></geometry>
       </collision>
     </link>
@@ -39,5 +39,5 @@
     <parent link="ur5_link1"/>
     <child link="ur5_link2"/>
-    <origin xyz="0 0 0.1200" rpy="0 0 0"/>
+    <origin xyz="0 0 0.0220" rpy="0 0 0"/>
     <axis xyz="0 1 0"/>
     <limit lower="-3.14159" upper="3.14159" effort="2.0" velocity="3.0"/>
@@ -48,5 +48,5 @@
     <parent link="ur5_link2"/>
     <child link="ur5_link3"/>
-    <origin xyz="0 0 0.1200" rpy="0 0 0"/>
+    <origin xyz="0 0 0.0220" rpy="0 0 0"/>
     <axis xyz="0 1 0"/>
     <limit lower="-3.14159" upper="3.14159" effort="2.0" velocity="3.0"/>
@@ -57,5 +57,5 @@
     <parent link="ur5_link3"/>
     <child link="ur5_link4"/>
-    <origin xyz="0 0 0.1200" rpy="0 0 0"/>
+    <origin xyz="0 0 0.0220" rpy="0 0 0"/>
     <axis xyz="0 1 0"/>
     <limit lower="-3.14159" upper="3.14159" effort="2.0" velocity="3.0"/>
@@ -66,5 +66,5 @@
     <parent link="ur5_link4"/>
     <child link="ur5_link5"/>
-    <origin xyz="0 0 0.1200" rpy="0 0 0"/>
+    <origin xyz="0 0 0.0220" rpy="0 0 0"/>
     <axis xyz="0 1 0"/>
     <limit lower="-3.14159" upper="3.14159" effort="2.0" velocity="3.0"/>
@@ -75,5 +75,5 @@
     <parent link="ur5_link5"/>
     <child link="ur5_link6"/>
-    <origin xyz="0 0 0.1200" rpy="0 0 0"/>
+    <origin xyz="0 0 0.0220" rpy="0 0 0"/>
     <axis xyz="0 1 0"/>
     <limit lower="-3.14159" upper="3.14159" effort="2.0" velocity="3.0"/>
@@ -94,5 +94,5 @@
     <parent link="ur5_link6"/>
     <child link="tool0"/>
-    <origin xyz="0 0 0.1300" rpy="0 0 0"/>
+    <origin xyz="0 0 0.0320" rpy="0 0 0"/>
   </joint>
   <xacro:arg name="sim_mode" default="gz"/>
