Commit message: Arm URDFs: add the mount transform so TF and MoveIt match Gazebo
The composed Gazebo models hang each arm 5 cm below base_link, flipped by
roll = pi (models/x500_with_<arm>/model.sdf, asset.yaml mount_*), but the
xacro URDFs that robot_state_publisher and MoveIt read attached the first
joint at base_link with no rotation. TF therefore drew every arm pointing
up, 0.33 m away from where the simulated end effector actually was, and
MoveIt planned for that arm. three_dof also placed ee_link 0.034 m past the
wrist where the SDF has 0.05 m.

uavros2/arm_kinematics.py computes end-effector forward kinematics from a
URDF and from a composed model SDF; test/test_arm_kinematics.py checks
both agree (position and orientation, 21 joint configurations per arm) and
that each arm's zero pose hangs between base_link and the gear feet.

File: arms/openmanip_x/urdf/openmanip_x.urdf.xacro (robot description, xacro)
@@ -30,5 +30,7 @@
     <parent link="base_link"/>
     <child link="openmanip_x_link1"/>
-    <origin xyz="0 0 0" rpy="0 0 0"/>
+    <!-- Mount: 5 cm below base_link, flipped (roll = pi) so the chain hangs
+         down; must match models/<uav>/model.sdf and asset.yaml mount_*. -->
+    <origin xyz="0 0 -0.05" rpy="3.14159 0 0"/>
     <axis xyz="0 1 0"/>
     <limit lower="-3.14159" upper="3.14159" effort="2.0" velocity="3.0"/>

File: arms/panda/urdf/panda.urdf.xacro (robot description, xacro)
@@ -30,5 +30,7 @@
     <parent link="base_link"/>
     <child link="panda_link1"/>
-    <origin xyz="0 0 0" rpy="0 0 0"/>
+    <!-- Mount: 5 cm below base_link, flipped (roll = pi) so the chain hangs
+         down; must match models/<uav>/model.sdf and asset.yaml mount_*. -->
+    <origin xyz="0 0 -0.05" rpy="3.14159 0 0"/>
     <axis xyz="0 1 0"/>
     <limit lower="-3.14159" upper="3.14159" effort="2.0" velocity="3.0"/>

File: arms/three_dof/urdf/three_dof.urdf.xacro (robot description, xacro)
@@ -58,5 +58,7 @@
     <parent link="base_link"/>
     <child link="shoulder_link"/>
-    <origin xyz="0 0 0.02" rpy="0 0 0"/>
+    <!-- Mount: 5 cm below base_link, flipped (roll = pi) so the chain hangs
+         down; must match models/<uav>/model.sdf and asset.yaml mount_*. -->
+    <origin xyz="0 0 -0.05" rpy="3.14159 0 0"/>
     <axis xyz="0 1 0"/>
     <limit lower="${-pi}" upper="${pi}" effort="2.0" velocity="3.0"/>
@@ -94,5 +96,5 @@
     <parent link="forearm_link"/>
     <child link="ee_link"/>
-    <origin xyz="0 0 ${link_len * 0.6 + 0.01}" rpy="0 0 0"/>
+    <origin xyz="0 0 0.05" rpy="0 0 0"/>
   </joint>
   <link name="ee_link">

File: arms/ur5/urdf/ur5.urdf.xacro (robot description, xacro)
@@ -30,5 +30,7 @@
     <parent link="base_link"/>
     <child link="ur5_link1"/>
-    <origin xyz="0 0 0" rpy="0 0 0"/>
+    <!-- Mount: 5 cm below base_link, flipped (roll = pi) so the chain hangs
+         down; must match models/<uav>/model.sdf and asset.yaml mount_*. -->
+    <origin xyz="0 0 -0.05" rpy="3.14159 0 0"/>
     <axis xyz="0 1 0"/>
     <limit lower="-3.14159" upper="3.14159" effort="2.0" velocity="3.0"/>

Commit message: OpenManipulator-X: real kinematics, masses and inertias (was a scaffold)
The openmanip_x arm was a 0.16 kg planar cylinder chain carrying the
ROBOTIS joint names. It now uses the upstream values from
ROBOTIS-GIT/open_manipulator (Apache-2.0): joint1 yaw and joints 2-4 pitch
at the real offsets, link masses/CoMs/inertias (0.594 kg total, gripper
fingers folded into the wrist), the real joint limits, and a 4.1 N m effort
limit (XM430-W350 stall torque). Geometry is boxes, not the STL meshes, and
there is no runtime dependency on the ROBOTIS packages. The joint names are
unchanged, so controllers.yaml keeps working.

Straight down the arm would reach 0.45 m, past the x500 gear feet
(-0.2195 m), so it spawns folded: ros2_control initial_value on the
position state interfaces (stow: joint2 -1.5, joint3 1.4, joint4 1.5),
which gz_ros2_control applies at startup. The SRDF home state is the stow
pose, KDL solves position-only IK, the airframe's hover thrust is 0.72.

models/x500_with_openmanip_x/model.sdf is generated from the xacro output;
test_arm_kinematics.py checks URDF and SDF agree and now checks each arm's
spawn pose (initial_value, else zero) above the landing gear instead of the
zero pose. aerial_arm_demo gets OMX poses for the real arm (forward reach,
side reach, fold, stow).

arms/mounts/*.urdf.xacro are removed: nothing loaded them, they included a
models/x500/urdf/x500.urdf.xacro that does not exist, and with the mount
inside each arm URDF they would apply it twice. The registry test now
checks each arm has a composed Gazebo model instead.

Verified: the arm spawns stowed, and 7 flights (2 s and 6 s arm motions)
take off, run all four poses and land.

File: arms/openmanip_x/urdf/openmanip_x.urdf.xacro (robot description, xacro)
@@ -1,31 +1,64 @@
 <?xml version="1.0"?>
 <!--
-  Scaffold URDF/Xacro for the openmanip_x arm: cylinder chain with the upstream
-  arm's joint names. Pairs with models/x500_with_openmanip_x/model.sdf so
-  ros2_control sees the same kinematics in Gazebo.
+  ROBOTIS OpenManipulator-X, mounted under the x500 (hangs below base_link).
+  Kinematics, masses, centres of mass, inertias and joint limits are the
+  upstream values from ROBOTIS-GIT/open_manipulator (Apache-2.0,
+  open_manipulator_description/urdf/open_manipulator_x/open_manipulator_x_arm.urdf.xacro):
+    joint1  yaw   (Z)  0.012 m along X from the base plate
+    joint2  pitch (Y)  0.0595 m above joint1
+    joint3  pitch (Y)  (0.024, 0, 0.128) from joint2
+    joint4  pitch (Y)  0.124 m along X from joint3
+    end_effector       0.126 m along X from joint4
+  Total arm mass 0.594 kg (the gripper fingers' 2 g are folded into link5;
+  the fingers themselves are not modelled). Visual / collision geometry is
+  boxes sized to each link instead of the upstream STL meshes.
+  Effort limit 4.1 N m: Dynamixel XM430-W350 stall torque at 12 V.
+  Pairs with models/x500_with_openmanip_x/model.sdf (test_arm_kinematics.py
+  checks they agree). The arm starts folded in the stow pose (initial_value
+  below) because straight down it would reach 0.45 m, past the landing gear.
 -->
 <robot xmlns:xacro="http://www.ros.org/wiki/xacro" name="openmanip_x">
-  <xacro:macro name="scaffold_link" params="name color_r color_g color_b">
+  <!-- Stow pose: upper arm swung back, forearm folded forward; every point of
+       the arm stays above z = -0.17 m (gear feet at -0.2195 m). -->
+  <xacro:property name="stow_j1" value="0.0"/>
+  <xacro:property name="stow_j2" value="-1.5"/>
+  <xacro:property name="stow_j3" value="1.4"/>
+  <xacro:property name="stow_j4" value="1.5"/>
+  <xacro:macro name="omx_link" params="name mass com ixx iyy izz ixy ixz iyz box box_xyz rgba">
     <link name="${name}">
       <inertial>
-        <mass value="0.04"/>
-        <origin xyz="0 0 0.0165" rpy="0 0 0"/>
-        <inertia ixx="4.270000e-06" iyy="4.270000e-06" izz="1.280000e-06"
-                 ixy="0" ixz="0" iyz="0"/>
+        <mass value="${mass}"/>
+        <origin xyz="${com}" rpy="0 0 0"/>
+        <inertia ixx="${ixx}" iyy="${iyy}" izz="${izz}" ixy="${ixy}" ixz="${ixz}" iyz="${iyz}"/>
       </inertial>
       <visual>
-        <origin xyz="0 0 0.0165" rpy="0 0 0"/>
-        <geometry><cylinder radius="0.008" length="0.033"/></geometry>
-        <material name="${name}_mat"><color rgba="${color_r} ${color_g} ${color_b} 1"/></material>
+        <origin xyz="${box_xyz}" rpy="0 0 0"/>
+        <geometry><box size="${box}"/></geometry>
+        <material name="${name}_mat"><color rgba="${rgba}"/></material>
       </visual>
       <collision>
-        <origin xyz="0 0 0.0165" rpy="0 0 0"/>
-        <geometry><cylinder radius="0.008" length="0.033"/></geometry>
+        <origin xyz="${box_xyz}" rpy="0 0 0"/>
+        <geometry><box size="${box}"/></geometry>
       </collision>
     </link>
   </xacro:macro>
+  <xacro:macro name="omx_joint" params="name parent child xyz axis lower upper">
+    <joint name="${name}" type="revolute">
+      <parent link="${parent}"/>
+      <child link="${child}"/>
+      <origin xyz="${xyz}" rpy="0 0 0"/>
+      <axis xyz="${axis}"/>
+      <limit lower="${lower}" upper="${upper}" effort="4.1" velocity="4.8"/>
+      <dynamics damping="0.05" friction="0.01"/>
+    </joint>
+  </xacro:macro>
   <link name="base_link"/>
-  <xacro:scaffold_link name="openmanip_x_link1" color_r="0.8" color_g="0.3" color_b="0.3"/>
-  <joint name="joint1" type="revolute">
+  <!-- Base plate, fixed to the drone. -->
+  <xacro:omx_link name="openmanip_x_link1" mass="7.9119962e-02"
+      com="3.0876154e-04 0 -1.2176461e-04"
+      ixx="1.2505234e-05" iyy="2.1898364e-05" izz="1.9267361e-05"
+      ixy="0" ixz="-1.7855208e-07" iyz="0"
+      box="0.045 0.045 0.017" box_xyz="0.012 0 0.0085" rgba="0.25 0.25 0.25 1"/>
+  <joint name="arm_mount" type="fixed">
     <parent link="base_link"/>
     <child link="openmanip_x_link1"/>
@@ -33,52 +66,59 @@
          down; must match models/<uav>/model.sdf and asset.yaml mount_*. -->
     <origin xyz="0 0 -0.05" rpy="3.14159 0 0"/>
-    <axis xyz="0 1 0"/>
-    <limit lower="-3.14159" upper="3.14159" effort="2.0" velocity="3.0"/>
-    <dynamics damping="0.05" friction="0.01"/>
   </joint>
-  <xacro:scaffold_link name="openmanip_x_link2" color_r="0.3" color_g="0.8" color_b="0.3"/>
-  <joint name="joint2" type="revolute">
-    <parent link="openmanip_x_link1"/>
-    <child link="openmanip_x_link2"/>
-    <origin xyz="0 0 0.0330" rpy="0 0 0"/>
-    <axis xyz="0 1 0"/>
-    <limit lower="-3.14159" upper="3.14159" effort="2.0" velocity="3.0"/>
-    <dynamics damping="0.05" friction="0.01"/>
-  </joint>
-  <xacro:scaffold_link name="openmanip_x_link3" color_r="0.3" color_g="0.3" color_b="0.8"/>
-  <joint name="joint3" type="revolute">
-    <parent link="openmanip_x_link2"/>
-    <child link="openmanip_x_link3"/>
-    <origin xyz="0 0 0.0330" rpy="0 0 0"/>
-    <axis xyz="0 1 0"/>
-    <limit lower="-3.14159" upper="3.14159" effort="2.0" velocity="3.0"/>
-    <dynamics damping="0.05" friction="0.01"/>
-  </joint>
-  <xacro:scaffold_link name="openmanip_x_link4" color_r="0.8" color_g="0.8" color_b="0.3"/>
-  <joint name="joint4" type="revolute">
-    <parent link="openmanip_x_link3"/>
-    <child link="openmanip_x_link4"/>
-    <origin xyz="0 0 0.0330" rpy="0 0 0"/>
-    <axis xyz="0 1 0"/>
-    <limit lower="-3.14159" upper="3.14159" effort="2.0" velocity="3.0"/>
-    <dynamics damping="0.05" friction="0.01"/>
-  </joint>
+  <xacro:omx_link name="openmanip_x_link2" mass="9.8406837e-02"
+      com="-3.0184870e-04 5.4043684e-04 4.7433464e-02"
+      ixx="3.4543422e-05" iyy="3.2689329e-05" izz="1.8850320e-05"
+      ixy="-1.6031095e-08" ixz="-3.8375155e-07" iyz="2.8511935e-08"
+      box="0.03 0.045 0.0595" box_xyz="0 0 0.03" rgba="0.85 0.85 0.85 1"/>
+  <xacro:omx_joint name="joint1" parent="openmanip_x_link1" child="openmanip_x_link2"
+      xyz="0.012 0 0" axis="0 0 1" lower="-3.14159" upper="3.14159"/>
+  <xacro:omx_link name="openmanip_x_link3" mass="1.3850917e-01"
+      com="1.0308393e-02 3.7743363e-04 1.0170197e-01"
+      ixx="3.3055381e-04" iyy="3.4290447e-04" izz="6.0346498e-05"
+      ixy="-9.7940978e-08" ixz="-3.8505711e-05" iyz="-1.5717516e-06"
+      box="0.035 0.03 0.15" box_xyz="0.012 0 0.064" rgba="0.25 0.25 0.25 1"/>
+  <xacro:omx_joint name="joint2" parent="openmanip_x_link2" child="openmanip_x_link3"
+      xyz="0 0 0.0595" axis="0 1 0" lower="-1.5" upper="1.5"/>
+  <xacro:omx_link name="openmanip_x_link4" mass="1.3274562e-01"
+      com="9.0909590e-02 3.8929816e-04 2.2413279e-04"
+      ixx="3.0654178e-05" iyy="2.4230292e-04" izz="2.5155057e-04"
+      ixy="-1.2764155e-06" ixz="-2.6874417e-07" iyz="1.1559550e-08"
+      box="0.124 0.03 0.03" box_xyz="0.062 0 0" rgba="0.85 0.85 0.85 1"/>
+  <xacro:omx_joint name="joint3" parent="openmanip_x_link3" child="openmanip_x_link4"
+      xyz="0.024 0 0.128" axis="0 1 0" lower="-1.5" upper="1.4"/>
+  <!-- Wrist + gripper (fingers' mass included). -->
+  <xacro:omx_link name="openmanip_x_link5" mass="1.4527573e-01"
+      com="4.4206755e-02 3.6839985e-07 8.9142216e-03"
+      ixx="8.0870749e-05" iyy="7.5980465e-05" izz="9.3127351e-05"
+      ixy="0" ixz="-1.0157896e-06" iyz="0"
+      box="0.10 0.05 0.03" box_xyz="0.05 0 0" rgba="0.25 0.25 0.25 1"/>
+  <xacro:omx_joint name="joint4" parent="openmanip_x_link4" child="openmanip_x_link5"
+      xyz="0.124 0 0" axis="0 1 0" lower="-1.7" upper="1.97"/>
   <link name="end_effector_link">
     <inertial>
-      <mass value="0.02"/>
-      <inertia ixx="1e-5" iyy="1e-5" izz="1e-5" ixy="0" ixz="0" iyz="0"/>
+      <mass value="0.001"/>
+      <inertia ixx="1e-8" iyy="1e-8" izz="1e-8" ixy="0" ixz="0" iyz="0"/>
     </inertial>
     <visual>
-      <geometry><sphere radius="0.018"/></geometry>
+      <geometry><sphere radius="0.01"/></geometry>
       <material name="ee_mat"><color rgba="1 1 0 1"/></material>
     </visual>
-    <collision><geometry><sphere radius="0.018"/></geometry></collision>
   </link>
   <joint name="j_ee" type="fixed">
-    <parent link="openmanip_x_link4"/>
+    <parent link="openmanip_x_link5"/>
     <child link="end_effector_link"/>
-    <origin xyz="0 0 0.0430" rpy="0 0 0"/>
+    <origin xyz="0.126 0 0" rpy="0 0 0"/>
   </joint>
   <xacro:arg name="sim_mode" default="gz"/>
+  <xacro:macro name="omx_control_joint" params="name initial">
+    <joint name="${name}">
+      <command_interface name="position"/>
+      <state_interface name="position">
+        <param name="initial_value">${initial}</param>
+      </state_interface>
+      <state_interface name="velocity"/>
+    </joint>
+  </xacro:macro>
   <ros2_control name="openmanip_x_hw" type="system">
     <hardware>
@@ -90,24 +130,8 @@
       </xacro:unless>
     </hardware>
-    <joint name="joint1">
-      <command_interface name="position"/>
-      <state_interface name="position"/>
-      <state_interface name="velocity"/>
-    </joint>
-    <joint name="joint2">
-      <command_interface name="position"/>
-      <state_interface name="position"/>
-      <state_interface name="velocity"/>
-    </joint>
-    <joint name="joint3">
-      <command_interface name="position"/>
-      <state_interface name="position"/>
-      <state_interface name="velocity"/>
-    </joint>
-    <joint name="joint4">
-      <command_interface name="position"/>
-      <state_interface name="position"/>
-      <state_interface name="velocity"/>
-    </joint>
+    <xacro:omx_control_joint name="joint1" initial="${stow_j1}"/>
+    <xacro:omx_control_joint name="joint2" initial="${stow_j2}"/>
+    <xacro:omx_control_joint name="joint3" initial="${stow_j3}"/>
+    <xacro:omx_control_joint name="joint4" initial="${stow_j4}"/>
   </ros2_control>
 </robot>

Commit message: OpenManipulator-X: collision-free stow pose; MoveIt plans and executes
The first stow pose (joint2 -1.5, joint3 1.4, joint4 1.5) folded the wrist
into the base links, so MoveIt rejected every request with
START_STATE_IN_COLLISION. The new stow (-1.1, 1.2, 0.9), found by a grid
search over the link boxes, has no self-contact, keeps the lowest point
1.6 cm above the gear feet and puts the arm's centre of mass under the
mount (no static pitch moment in hover). The demo's third pose swings the
arm back (CoM 0.13 m behind the mount, mirroring the forward reach)
instead of a fold that also self-collided.

All four SRDFs declared the arm group as its own end effector's parent,
which MoveIt rejects ("cannot be its own parent"); the element is removed
until there is a gripper group.

Verified with use_moveit:=true: plans to the forward, side and backward
reaches succeed, and a planned joint1 move executes through
joint_trajectory_controller (0.597 rad for a 0.6 rad goal) and back.

File: arms/openmanip_x/urdf/openmanip_x.urdf.xacro (robot description, xacro)
@@ -19,10 +19,12 @@
 -->
 <robot xmlns:xacro="http://www.ros.org/wiki/xacro" name="openmanip_x">
-  <!-- Stow pose: upper arm swung back, forearm folded forward; every point of
-       the arm stays above z = -0.17 m (gear feet at -0.2195 m). -->
+  <!-- Stow pose: upper arm swung back, forearm and wrist folded forward. The
+       arm's centre of mass sits right under the mount (no static pitch
+       moment), its lowest point is 1.6 cm above the gear feet (-0.2195 m),
+       and no two non-adjacent links touch, so MoveIt can plan from it. -->
   <xacro:property name="stow_j1" value="0.0"/>
-  <xacro:property name="stow_j2" value="-1.5"/>
-  <xacro:property name="stow_j3" value="1.4"/>
-  <xacro:property name="stow_j4" value="1.5"/>
+  <xacro:property name="stow_j2" value="-1.1"/>
+  <xacro:property name="stow_j3" value="1.2"/>
+  <xacro:property name="stow_j4" value="0.9"/>
   <xacro:macro name="omx_link" params="name mass com ixx iyy izz ixy ixz iyz box box_xyz rgba">
     <link name="${name}">

Commit message: Contact tool, wall world and wall_contact_demo
x500_with_openmanip_x_tool: OMX plus a 0.40 m rod with a force/torque sensor
(airframe 4029); worlds/wall.sdf has a wall at x = 3 m. wall_contact_demo flies
to the wall, presses under plain position control and logs force and tip
position. Tests check the tool's URDF/SDF kinematics and stow clearance.

File: arms/openmanip_x/urdf/openmanip_x.urdf.xacro (robot description, xacro)
@@ -23,8 +23,13 @@
        moment), its lowest point is 1.6 cm above the gear feet (-0.2195 m),
        and no two non-adjacent links touch, so MoveIt can plan from it. -->
+  <xacro:arg name="tool" default="none"/>
+  <xacro:property name="has_tool" value="${'$(arg tool)' == 'rod'}"/>
   <xacro:property name="stow_j1" value="0.0"/>
-  <xacro:property name="stow_j2" value="-1.1"/>
-  <xacro:property name="stow_j3" value="1.2"/>
-  <xacro:property name="stow_j4" value="0.9"/>
+  <!-- With the 0.40 m contact tool that pose puts the rod through the frame;
+       this one points the rod backwards under the body, above the gear feet,
+       with no static pitch moment. -->
+  <xacro:property name="stow_j2" value="${0.9 if has_tool else -1.1}"/>
+  <xacro:property name="stow_j3" value="${1.1 if has_tool else 1.2}"/>
+  <xacro:property name="stow_j4" value="${1.3 if has_tool else 0.9}"/>
   <xacro:macro name="omx_link" params="name mass com ixx iyy izz ixy ixz iyz box box_xyz rgba">
     <link name="${name}">
@@ -113,4 +118,32 @@
     <origin xyz="0.126 0 0" rpy="0 0 0"/>
   </joint>
+  <xacro:if value="${has_tool}">
+    <!-- Contact tool, as in models/x500_with_openmanip_x_tool/model.sdf. -->
+    <link name="tool_link">
+      <inertial>
+        <origin xyz="0.2 0 0"/>
+        <mass value="0.12"/>
+        <inertia ixx="2e-6" iyy="1.6e-3" izz="1.6e-3" ixy="0" ixz="0" iyz="0"/>
+      </inertial>
+      <visual>
+        <origin xyz="0.2 0 0" rpy="0 1.5708 0"/>
+        <geometry><cylinder radius="0.006" length="0.4"/></geometry>
+      </visual>
+      <collision>
+        <origin xyz="0.4 0 0"/>
+        <geometry><sphere radius="0.015"/></geometry>
+      </collision>
+    </link>
+    <joint name="j_tool" type="fixed">
+      <parent link="end_effector_link"/>
+      <child link="tool_link"/>
+    </joint>
+    <link name="tool_tip"/>
+    <joint name="j_tool_tip" type="fixed">
+      <parent link="tool_link"/>
+      <child link="tool_tip"/>
+      <origin xyz="0.4 0 0"/>
+    </joint>
+  </xacro:if>
   <xacro:arg name="sim_mode" default="gz"/>
   <xacro:macro name="omx_control_joint" params="name initial">

Commit message: Contact tool: two-point head; compensation and contact results
Pushed against a wall, a single-point tool buckles in yaw and the drone falls.
A 0.20 m two-point head helps at 3 N, not at 6 N. docs/AERIAL_ARM.md has the
feed-forward comparison (at 2 s motions the worst peak falls from 50 cm to 19 cm
with the outer loop, 13 cm with the PX4 patch) and the contact tables.

File: arms/openmanip_x/urdf/openmanip_x.urdf.xacro (robot description, xacro)
@@ -130,6 +130,14 @@
         <geometry><cylinder radius="0.006" length="0.4"/></geometry>
       </visual>
+      <visual>
+        <origin xyz="0.4 0 0" rpy="1.5708 0 0"/>
+        <geometry><cylinder radius="0.015" length="0.2"/></geometry>
+      </visual>
       <collision>
-        <origin xyz="0.4 0 0"/>
+        <origin xyz="0.4 0.1 0"/>
+        <geometry><sphere radius="0.015"/></geometry>
+      </collision>
+      <collision>
+        <origin xyz="0.4 -0.1 0"/>
         <geometry><sphere radius="0.015"/></geometry>
       </collision>

Commit message: Contact on simulated RTK: pivot on the body's axis, longer rod; failed starts explained
Tool: 0.50 m rod, arm folded so the yaw pivot sits on the body's axis, softer spring.
With RTK through PX4's EKF, 9 of 10 runs hold 3 N for 60 s, tool height SD 2-6 cm
against 13-26 cm on plain GPS. The target of 10 of 10 within 2 cm is not met, and 6 N
is not held. The arm's correction in the air makes things worse on RTK. Failed starts
are machine load, not GPS: 18 of 18 fine at load 3-20.

File: arms/openmanip_x/urdf/openmanip_x.urdf.xacro (robot description, xacro)
@@ -26,5 +26,5 @@
   <xacro:property name="has_tool" value="${'$(arg tool)' == 'rod'}"/>
   <xacro:property name="stow_j1" value="0.0"/>
-  <!-- With the 0.40 m contact tool that pose puts the rod through the frame;
+  <!-- With the 0.50 m contact tool that pose puts the rod through the frame;
        this one points the rod backwards under the body, above the gear feet,
        with no static pitch moment. -->
@@ -122,22 +122,22 @@
     <link name="tool_link">
       <inertial>
-        <origin xyz="0.2 0 0"/>
-        <mass value="0.12"/>
-        <inertia ixx="2e-6" iyy="1.6e-3" izz="1.6e-3" ixy="0" ixz="0" iyz="0"/>
+        <origin xyz="0.26 0 0"/>
+        <mass value="0.14"/>
+        <inertia ixx="2e-6" iyy="2.9e-3" izz="2.9e-3" ixy="0" ixz="0" iyz="0"/>
       </inertial>
       <visual>
-        <origin xyz="0.2 0 0" rpy="0 1.5708 0"/>
-        <geometry><cylinder radius="0.006" length="0.4"/></geometry>
+        <origin xyz="0.25 0 0" rpy="0 1.5708 0"/>
+        <geometry><cylinder radius="0.006" length="0.5"/></geometry>
       </visual>
       <visual>
-        <origin xyz="0.4 0 0" rpy="1.5708 0 0"/>
+        <origin xyz="0.5 0 0" rpy="1.5708 0 0"/>
         <geometry><cylinder radius="0.015" length="0.2"/></geometry>
       </visual>
       <collision>
-        <origin xyz="0.4 0.1 0"/>
+        <origin xyz="0.5 0.1 0"/>
         <geometry><sphere radius="0.015"/></geometry>
       </collision>
       <collision>
-        <origin xyz="0.4 -0.1 0"/>
+        <origin xyz="0.5 -0.1 0"/>
         <geometry><sphere radius="0.015"/></geometry>
       </collision>
@@ -151,5 +151,5 @@
       <parent link="tool_link"/>
       <child link="tool_tip"/>
-      <origin xyz="0.4 0 0"/>
+      <origin xyz="0.5 0 0"/>
     </joint>
   </xacro:if>
