Commit message: three_dof arm: end-to-end Gazebo + MoveIt + cosmetic cleanups
models/x500_with_three_dof_arm/{model.sdf,model.config}:
  Composed SDF including x500 base + 3-DOF arm links/joints +
  gz_ros2_control plugin. Mirrors the URDF dimensions exactly.

arms/three_dof/urdf/three_dof.urdf.xacro:
  Added <ros2_control> block with sim_mode xacro arg
  (gz -> GazeboSimSystem, otherwise mock_components/GenericSystem)
  so the same xacro is reusable across simulators.

arms/three_dof/config/moveit/:
  SRDF, kinematics.yaml, ompl_planning.yaml,
  moveit_controllers.yaml, joint_limits.yaml. Minimal but
  functional config for the 3-DOF planning group.

arms/three_dof/asset.yaml: moveit: true, plus moveit_group and
  moveit_ee_link metadata for downstream tooling.

launch/arm_control.launch.py:
  - Expands xacro with sim_mode appropriate for the current simulator
  - Spawns robot_state_publisher with the URDF (gz_ros2_control
    reads it from there)
  - Delays spawner Nodes a few seconds so the controller_manager
    (hosted by gz_ros2_control) has time to come up
  - When use_moveit:=true, loads all five MoveIt YAMLs into
    move_group, with a longer delay so controllers are spawned first

launch/sim_common.launch.py + launch/simulators/gazebo.launch.py:
  Switch static_transform_publisher Nodes to the new-style named
  args (--x --y --z --yaw --pitch --roll --frame-id
  --child-frame-id) to silence the "Old-style arguments are
  deprecated" warnings.

Known-benign warning (not addressed; upstream mavros):
  /drone/mavros/global_position/gp_origin RELIABILITY QoS mismatch
  between mavros' own global_position publisher and guided_target
  subscriber. Internal to mavros, no impact on canonical topics.

File: arms/three_dof/urdf/three_dof.urdf.xacro (robot description, xacro)
@@ -90,3 +90,36 @@
     <collision><geometry><sphere radius="0.015"/></geometry></collision>
   </link>
+  <!--
+    ros2_control hardware interface. Same xacro is consumed by:
+    - Gazebo (via gz_ros2_control plugin in the composed model.sdf):
+      uses gz_ros2_control/GazeboSimSystem
+    - Other simulators / mock hardware: uses mock_components/GenericSystem
+    The xacro:arg `sim_mode` toggles between the two; defaults to gz.
+  -->
+  <xacro:arg name="sim_mode" default="gz"/>
+  <ros2_control name="three_dof_hw" type="system">
+    <hardware>
+      <xacro:if value="${'$(arg sim_mode)' == 'gz'}">
+        <plugin>gz_ros2_control/GazeboSimSystem</plugin>
+      </xacro:if>
+      <xacro:unless value="${'$(arg sim_mode)' == 'gz'}">
+        <plugin>mock_components/GenericSystem</plugin>
+      </xacro:unless>
+    </hardware>
+    <joint name="j_shoulder">
+      <command_interface name="position"/>
+      <state_interface name="position"/>
+      <state_interface name="velocity"/>
+    </joint>
+    <joint name="j_elbow">
+      <command_interface name="position"/>
+      <state_interface name="position"/>
+      <state_interface name="velocity"/>
+    </joint>
+    <joint name="j_wrist">
+      <command_interface name="position"/>
+      <state_interface name="position"/>
+      <state_interface name="velocity"/>
+    </joint>
+  </ros2_control>
 </robot>

Commit message: Docs sync to reality + silence kdl_parser root-inertia warning
docs/MANIPULATORS.md:
  - Strip stale claims that scaffolds require upstream description
    packages installed (the scaffolds are self-contained cylinder
    chains; they just borrow the upstream joint-name conventions).
  - Document the gear-fit budget (drop <= 0.20 m below base_link).
  - Document the per-arm drop and gear-feet margin (21-34 mm above).
  - Document the use_moveit dispatcher arg.
  - List joint names per arm for the action send_goal examples.
  - Add a "Replacing a scaffold with the real arm" section pointing
    at the upstream_pkg field in each asset.yaml.

docs/MODELS.md:
  - Add the four composed arm models (x500_with_three_dof_arm,
    _openmanip_x, _panda, _ur5) to the inventory table with their
    PX4 airframes (4025-4028).
  - Cross-reference MANIPULATORS.md for per-arm detail.

docs/SIMULATORS.md:
  - Mark gazebo as "Working end-to-end (PX4 + MAVROS +
    gz_ros2_control + MoveIt)" with all 4 arms.
  - Downgrade webots / mujoco from "Working" to "Scaffolded" - they
    have launch stubs but no real demo yet (was aspirational).
  - Fix the wrong gazebo launch example
    (uav:=x500_d435 arm:=panda doesn't work - need
    uav:=x500_with_panda). Add the with-arm form alongside.
  - Add the use_moveit:=true form.

arms/three_dof/urdf/three_dof.urdf.xacro:
  - Add a dummy world_link with no inertia + fixed joint to base_link.
  - Silences the recurring runtime warning:
      [kdl_parser]: The root link base_link has an inertia specified
      in the URDF, but KDL does not support a root link with an
      inertia.  As a workaround, you can add an extra dummy link to
      your URDF.
  - The three scaffold arms (openmanip_x, panda, ur5) had empty
    base_link by construction, so they didn't trigger the warning
    and don't need this fix.

42 pytest still green.

File: arms/three_dof/urdf/three_dof.urdf.xacro (robot description, xacro)
@@ -39,4 +39,16 @@
     </collision>
   </xacro:macro>
+  <!--
+    Dummy world_link with no inertia silences the kdl_parser warning:
+    "The root link base_link has an inertia specified in the URDF, but
+    KDL does not support a root link with an inertia." Fixed joint keeps
+    kinematics unchanged.
+  -->
+  <link name="world_link"/>
+  <joint name="world_to_base" type="fixed">
+    <parent link="world_link"/>
+    <child link="base_link"/>
+    <origin xyz="0 0 0" rpy="0 0 0"/>
+  </joint>
   <link name="base_link">
     <xacro:cyl_inertia m="0.05" r="0.02" l="0.02"/>
